File: connections/chimeraConn/chimeraConn.kicad_sch (KiCad schematic)
At the start: 5 parts, among them M1 SpeedyBee_Nano_2.4G, M2 camera, M3 Foxeer M10Q-120 compass, M4 Foxeer Reaper Nano V2 VTx 5.8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

Commit message: add technical drawing
Parts:
- M2: value camera -> Foxeer Cat 3 micro

Commit message: update for MkII release
Parts:
- M3: value Foxeer M10Q-120 compass -> Foxeer M10Q-180 compass
